Commit message: removed knuckle joint

File: urdf/ur.ros2_control.xacro (robot description, xacro)
@@ -55,4 +55,25 @@
         </xacro:unless>
       </hardware>
+ <!--     <joint name="robotiq_85_left_knuckle_joint">
+                <command_interface name="position" />
+                <command_interface name="velocity" />
+                <state_interface name="position">
+                  <param name="initial_value">0.0</param>
+                </state_interface>
+                <state_interface name="velocity"/>
+                <state_interface name="effort"/>
+      </joint>
+      <joint name="robotiq_85_right_knuckle_joint">
+                <param name="mimic">robotiq_85_left_knuckle_joint</param>
+                <param name="multiplier">1</param>
+                <command_interface name="position" />
+                <command_interface name="velocity" />
+                <state_interface name="position">
+                  <param name="initial_value">0.0</param>
+                </state_interface>
+                <state_interface name="velocity"/>
+                <state_interface name="effort"/>
+      </joint>
+-->
       <joint name="${prefix}shoulder_pan_joint">
         <command_interface name="position">

Commit message: gripper joints now in different hardware interface

File: urdf/ur.ros2_control.xacro (robot description, xacro)
@@ -17,4 +17,38 @@
     reverse_port:=50001
     script_sender_port:=50002">
+    <ros2_control name="${name}_gripper" type="system">
+      <hardware>
+        <xacro:if value="${sim_gazebo}">
+          <plugin>gazebo_ros2_control/GazeboSystem</plugin>
+        </xacro:if>
+        <xacro:if value="${sim_ignition}">
+          <plugin>ign_ros2_control/IgnitionSystem</plugin>
+        </xacro:if>
+        <xacro:if value="${use_fake_hardware}">
+          <plugin>fake_components/GenericSystem</plugin>
+          <param name="fake_sensor_commands">${fake_sensor_commands}</param>
+          <param name="state_following_offset">0.0</param>
+        </xacro:if>
+        <xacro:unless value="${use_fake_hardware or sim_gazebo or sim_ignition}">
+          <plugin>fake_components/GenericSystem</plugin>
+        </xacro:unless>
+      </hardware>
+      <joint name="robotiq_85_left_knuckle_joint">
+                <command_interface name="position" />
+                <state_interface name="position">
+                  <param name="initial_value">0.0</param>
+                </state_interface>
+                <state_interface name="velocity"/>
+      </joint>
+      <joint name="robotiq_85_right_knuckle_joint">
+                <param name="mimic">robotiq_85_left_knuckle_joint</param>
+                <param name="multiplier">1</param>
+                <command_interface name="position" />
+                <state_interface name="position">
+                  <param name="initial_value">0.0</param>
+                </state_interface>
+                <state_interface name="velocity"/>
+      </joint>
+    </ros2_control>
     <ros2_control name="${name}" type="system">
       <hardware>
@@ -55,25 +89,4 @@
         </xacro:unless>
       </hardware>
- <!--     <joint name="robotiq_85_left_knuckle_joint">
-                <command_interface name="position" />
-                <command_interface name="velocity" />
-                <state_interface name="position">
-                  <param name="initial_value">0.0</param>
-                </state_interface>
-                <state_interface name="velocity"/>
-                <state_interface name="effort"/>
-      </joint>
-      <joint name="robotiq_85_right_knuckle_joint">
-                <param name="mimic">robotiq_85_left_knuckle_joint</param>
-                <param name="multiplier">1</param>
-                <command_interface name="position" />
-                <command_interface name="velocity" />
-                <state_interface name="position">
-                  <param name="initial_value">0.0</param>
-                </state_interface>
-                <state_interface name="velocity"/>
-                <state_interface name="effort"/>
-      </joint>
--->
       <joint name="${prefix}shoulder_pan_joint">
         <command_interface name="position">

Commit message: replaced urdf and meshes with the ones from picknik, fused them with ur urdf

File: urdf/ur.ros2_control.xacro (robot description, xacro)
@@ -17,5 +17,5 @@
     reverse_port:=50001
     script_sender_port:=50002">
-    <ros2_control name="${name}_gripper" type="system">
+ <!--   <ros2_control name="${name}_gripper" type="system">
       <hardware>
         <xacro:if value="${sim_gazebo}">
@@ -51,4 +51,5 @@
       </joint>
     </ros2_control>
+-->
     <ros2_control name="${name}" type="system">
       <hardware>

File: urdf/ur.urdf.xacro (robot description, xacro)
@@ -6,5 +6,5 @@
    <xacro:include filename="$(find ur_description)/urdf/ur_macro.xacro"/>
    <xacro:include filename="$(find ur_description)/urdf/table_macro.xacro"/>
-   <xacro:include filename="$(find ur_description)/urdf/robotiq_85_gripper_macro.urdf.xacro"/>
+   <xacro:include filename="$(find ur_description)/urdf/robotiq_gripper_macro.urdf.xacro"/>
    <!-- possible 'ur_type' values: ur3, ur3e, ur5, ur5e, ur10, ur10e, ur16e -->
    <!-- the default value should raise an error in case this was called without defining the type -->
@@ -93,10 +93,10 @@
    </xacro:table_attach>
    <!-- gripper -->
-   <xacro:robotiq_85_gripper
+   <xacro:robotiq_gripper
      prefix="$(arg prefix)"
      parent="tool0"
      >
-     <origin xyz="0.0 0.0 0.0" rpy="-1.57 -1.57 0"/>
-   </xacro:robotiq_85_gripper>
+     <origin xyz="0.0 0.0 0.0" rpy="0 0 0"/>
+   </xacro:robotiq_gripper>
    <!-- arm -->
    <xacro:ur_robot
