Commit message: Hide visual of wall and top, add colour to table

File: urdf/table_collision_macro.xacro (robot description, xacro)
@@ -3,5 +3,5 @@
   <xacro:include filename="$(find ur_description)/urdf/inc/model_common.xacro" />
   <xacro:include filename="$(find ur_description)/urdf/inc/table_common.xacro" />
-  <xacro:macro name="table_attach" params="
+  <xacro:macro name="table_collision_attach" params="
     prefix
     name
@@ -13,7 +13,4 @@
     physical_parameters_table_file
    ">
-  <material name="dullbrown" >
-    <color rgba="0.5294117647058824 0.43137254901960786 0.29411764705882354 1.0" />
-  </material>
   <!-- links -->
   <link name="${prefix}${name}_link">
@@ -21,7 +18,6 @@
       <origin rpy="0 0 0" xyz="0 0 ${-table_inertia_z/2}"/>
       <geometry>
-        <box size="${table_inertia_x} ${table_inertia_y} ${table_inertia_z}"/>
+        <box size="0 0 0"/>
       </geometry>
-      <material name="dullbrown"/>
     </visual>
     <collision>

File: urdf/ur.urdf.xacro (robot description, xacro)
@@ -6,4 +6,5 @@
    <xacro:include filename="$(find ur_description)/urdf/ur_macro.xacro"/>
    <xacro:include filename="$(find ur_description)/urdf/table_macro.xacro"/>
+   <xacro:include filename="$(find ur_description)/urdf/table_collision_macro.xacro"/>
    <xacro:include filename="$(find ur_description)/urdf/robotiq_gripper_macro.urdf.xacro"/>
    <!-- possible 'ur_type' values: ur3, ur3e, ur5, ur5e, ur10, ur10e, ur16e -->
@@ -73,5 +74,5 @@
    </xacro:table_attach>
    <!-- top -->
-   <xacro:table_attach
+   <xacro:table_collision_attach
      prefix="$(arg prefix)"
      name="top"
@@ -83,7 +84,7 @@
      >
      <origin xyz="-0.232 0.415 0.7" rpy="0 0 0"/>
-   </xacro:table_attach>
+   </xacro:table_collision_attach>
     <!-- wall -->
-   <xacro:table_attach
+   <xacro:table_collision_attach
      prefix="$(arg prefix)"
      name="wall"
@@ -95,5 +96,5 @@
      >
      <origin xyz="-0.618 0.0 0.35" rpy="0 1.57 0"/>
-   </xacro:table_attach>
+   </xacro:table_collision_attach>
    <!-- gripper -->
    <xacro:if value="$(arg use_gripper)">
