Commit message: Updated ringlight, beam,and wall models with visual.

File: urdf/beam_macro.xacro (robot description, xacro)
@@ -3,5 +3,5 @@
   <xacro:include filename="$(find ur_description)/urdf/inc/model_common.xacro" />
   <xacro:include filename="$(find ur_description)/urdf/inc/table_common.xacro" />
-  <xacro:macro name="table_collision_attach" params="
+  <xacro:macro name="beam_attach" params="
     prefix
     name
@@ -12,6 +12,8 @@
     gazebo_preserve_fixed_joint
     physical_parameters_table_file
-    collision_geometry
    ">
+  <material name="gunmetal" >
+    <color rgba="0.3254901960784314 0.3843137254901961 0.403921568627451 1.0" />
+  </material>
   <!-- links -->
   <link name="${prefix}${name}_link">
@@ -19,19 +21,15 @@
       <origin rpy="0 0 0" xyz="0 0 ${-table_inertia_z/2}"/>
       <geometry>
-        <box size="0 0 0"/>
+        <box size="${beam_inertia_x} ${beam_inertia_y} ${beam_inertia_z}"/>
       </geometry>
+      <material name="gunmetal"/>
     </visual>
     <collision>
       <origin rpy="0 0 0" xyz="0 0 ${-table_inertia_z/2}"/>
       <geometry>
-        <xacro:if value="${collision_geometry == 'box'}">
-          <box size="1.5 2.0 0.05"/>
-        </xacro:if>
-        <xacro:if value="${collision_geometry == 'cylinder'}">
-          <cylinder radius="0.3" length="0.03" />
-        </xacro:if>
+        <box size="${beam_inertia_x} ${beam_inertia_y} ${beam_inertia_z}"/>
       </geometry>
     </collision>
-    <xacro:box_inertial x="${table_inertia_x}" y="${table_inertia_y}" z="${table_inertia_z}"  m="${table_mass}">
+    <xacro:box_inertial x="${beam_inertia_x}" y="${beam_inertia_y}" z="${beam_inertia_z}"  m="${beam_mass}">
       <origin rpy="0 0 0" xyz="0 0 ${-table_inertia_z/2}"/>
     </xacro:box_inertial>

File: urdf/inc/model_common.xacro (robot description, xacro)
@@ -1,5 +1,5 @@
 <?xml version="1.0"?>
 <robot xmlns:xacro="http://wiki.ros.org/xacro">
-  <xacro:macro name="cylinder_inertial_model_common" params="radius length mass *origin">
+  <xacro:macro name="cylinder_inertial" params="radius length mass *origin">
     <inertial>
       <mass value="${mass}" />

File: urdf/inc/table_common.xacro (robot description, xacro)
@@ -8,4 +8,7 @@
     <!-- mass -->
     <xacro:property name="table_mass" value="${sec_inertia_parameters['table_mass']}" scope="parent"/>
+    <xacro:property name="beam_mass" value="${sec_inertia_parameters['beam_mass']}" scope="parent"/>
+    <xacro:property name="wall_mass" value="${sec_inertia_parameters['wall_mass']}" scope="parent"/>
+    <xacro:property name="ringlight_mass" value="${sec_inertia_parameters['ringlight_mass']}" scope="parent"/>
     <!-- dimensions -->
     <xacro:property name="inertia_links" value="${sec_inertia_parameters['links']}" scope="parent"/>
@@ -13,4 +16,12 @@
     <xacro:property name="table_inertia_y" value="${inertia_links['table']['y']}" scope="parent"/>
     <xacro:property name="table_inertia_z" value="${inertia_links['table']['z']}" scope="parent"/>
+    <xacro:property name="beam_inertia_x" value="${inertia_links['beam']['x']}" scope="parent"/>
+    <xacro:property name="beam_inertia_y" value="${inertia_links['beam']['y']}" scope="parent"/>
+    <xacro:property name="beam_inertia_z" value="${inertia_links['beam']['z']}" scope="parent"/>
+    <xacro:property name="wall_inertia_x" value="${inertia_links['wall']['x']}" scope="parent"/>
+    <xacro:property name="wall_inertia_y" value="${inertia_links['wall']['y']}" scope="parent"/>
+    <xacro:property name="wall_inertia_z" value="${inertia_links['wall']['z']}" scope="parent"/>
+    <xacro:property name="ringlight_inertia_radius" value="${inertia_links['ringlight']['radius']}" scope="parent"/>
+    <xacro:property name="ringlight_inertia_length" value="${inertia_links['ringlight']['length']}" scope="parent"/>
   </xacro:macro>
 </robot>

File: urdf/ringlight_macro.xacro (robot description, xacro)
@@ -3,5 +3,5 @@
   <xacro:include filename="$(find ur_description)/urdf/inc/model_common.xacro" />
   <xacro:include filename="$(find ur_description)/urdf/inc/table_common.xacro" />
-  <xacro:macro name="table_collision_attach" params="
+  <xacro:macro name="ringlight_attach" params="
     prefix
     name
@@ -12,6 +12,8 @@
     gazebo_preserve_fixed_joint
     physical_parameters_table_file
-    collision_geometry
    ">
+  <material name="palegrey" >
+    <color rgba="0.9921568627450981 0.9921568627450981 0.996078431372549 1.0" />
+  </material>
   <!-- links -->
   <link name="${prefix}${name}_link">
@@ -19,21 +21,17 @@
       <origin rpy="0 0 0" xyz="0 0 ${-table_inertia_z/2}"/>
       <geometry>
-        <box size="0 0 0"/>
+        <cylinder radius="${ringlight_inertia_radius}" length="${ringlight_inertia_length}" />
       </geometry>
+      <material name="palegrey"/>
     </visual>
     <collision>
       <origin rpy="0 0 0" xyz="0 0 ${-table_inertia_z/2}"/>
       <geometry>
-        <xacro:if value="${collision_geometry == 'box'}">
-          <box size="1.5 2.0 0.05"/>
-        </xacro:if>
-        <xacro:if value="${collision_geometry == 'cylinder'}">
-          <cylinder radius="0.3" length="0.03" />
-        </xacro:if>
+        <cylinder radius="${ringlight_inertia_radius}" length="${ringlight_inertia_length}" />
       </geometry>
     </collision>
-    <xacro:box_inertial x="${table_inertia_x}" y="${table_inertia_y}" z="${table_inertia_z}"  m="${table_mass}">
+    <xacro:cylinder_inertial radius="${ringlight_inertia_radius}" length="${ringlight_inertia_length}" mass="${ringlight_mass}" >
       <origin rpy="0 0 0" xyz="0 0 ${-table_inertia_z/2}"/>
-    </xacro:box_inertial>
+    </xacro:cylinder_inertial>
   </link>
   <xacro:if value="${sim_ignition}">

File: urdf/table_macro.xacro (robot description, xacro)
@@ -16,4 +16,7 @@
     <color rgba="0.5294117647058824 0.43137254901960786 0.29411764705882354 1.0" />
   </material>
+   <material name="orangeyellow" >
+    <color rgba="1.0 0.6784313725490196 0.00392156862745098 1.0" />
+  </material>
   <!-- links -->
   <link name="${prefix}${name}_link">
@@ -23,5 +26,5 @@
         <box size="${table_inertia_x} ${table_inertia_y} ${table_inertia_z}"/>
       </geometry>
-      <material name="dullbrown"/>
+      <material name="orangeyellow"/>
     </visual>
     <collision>

File: urdf/ur.urdf.xacro (robot description, xacro)
@@ -6,4 +6,7 @@
    <xacro:include filename="$(find ur_description)/urdf/ur_macro.xacro"/>
    <xacro:include filename="$(find ur_description)/urdf/table_macro.xacro"/>
+   <xacro:include filename="$(find ur_description)/urdf/beam_macro.xacro"/>
+   <xacro:include filename="$(find ur_description)/urdf/wall_macro.xacro"/>
+   <xacro:include filename="$(find ur_description)/urdf/ringlight_macro.xacro"/>
    <xacro:include filename="$(find ur_description)/urdf/table_collision_macro.xacro"/>
    <xacro:include filename="$(find ur_description)/urdf/robotiq_gripper_macro.urdf.xacro"/>
@@ -43,4 +46,5 @@
    <!-- Table parameters -->
    <xacro:arg name="physical_params_table" default="$(find ur_description)/config/table/physical_parameters_table.yaml"/>
+   <xacro:arg name="ring_beam_height" default="1.0"/>
      <!-- Simulation parameters -->
    <xacro:arg name="use_fake_hardware" default="false" />
@@ -75,8 +79,8 @@
      <origin xyz="-0.232 0.415 0" rpy="0 0 0"/>
    </xacro:table_attach>
-   <!-- top -->
-   <xacro:table_collision_attach
+   <!-- ringlight -->
+   <xacro:ringlight_attach
      prefix="$(arg prefix)"
-     name="top"
+     name="ringlight"
      parent="world"
      sim_gazebo="$(arg sim_gazebo)"
@@ -85,8 +89,20 @@
      physical_parameters_table_file="$(arg physical_params_table)"
      >
-     <origin xyz="-0.232 0.415 0.7" rpy="0 0 0"/>
-   </xacro:table_collision_attach>
+     <origin xyz="-0.232 0.415 $(arg ring_beam_height)" rpy="0 0 0"/>
+   </xacro:ringlight_attach>
+   <!-- beam -->
+   <xacro:beam_attach
+     prefix="$(arg prefix)"
+     name="beam"
+     parent="world"
+     sim_gazebo="$(arg sim_gazebo)"
+     sim_ignition="$(arg sim_ignition)"
+     gazebo_preserve_fixed_joint="$(arg gazebo_preserve_fixed_joint_arg)"
+     physical_parameters_table_file="$(arg physical_params_table)"
+     >
+     <origin xyz="-0.518 0.415 $(arg ring_beam_height)" rpy="0 0 0"/>
+   </xacro:beam_attach>
     <!-- wall -->
-   <xacro:table_collision_attach
+   <xacro:wall_attach
      prefix="$(arg prefix)"
      name="wall"
@@ -98,5 +114,5 @@
      >
      <origin xyz="-0.618 0.0 0.35" rpy="0 1.57 0"/>
-   </xacro:table_collision_attach>
+   </xacro:wall_attach>
    <!-- gripper -->
    <xacro:if value="$(arg use_gripper)">

File: urdf/wall_macro.xacro (robot description, xacro)
@@ -3,5 +3,5 @@
   <xacro:include filename="$(find ur_description)/urdf/inc/model_common.xacro" />
   <xacro:include filename="$(find ur_description)/urdf/inc/table_common.xacro" />
-  <xacro:macro name="table_collision_attach" params="
+  <xacro:macro name="wall_attach" params="
     prefix
     name
@@ -12,6 +12,8 @@
     gazebo_preserve_fixed_joint
     physical_parameters_table_file
-    collision_geometry
    ">
+  <material name="offwhite" >
+    <color rgba="1.0 1.0 0.8941176470588236 1.0" />
+  </material>
   <!-- links -->
   <link name="${prefix}${name}_link">
@@ -19,19 +21,15 @@
       <origin rpy="0 0 0" xyz="0 0 ${-table_inertia_z/2}"/>
       <geometry>
-        <box size="0 0 0"/>
+        <box size="${wall_inertia_x} ${wall_inertia_y} ${wall_inertia_z}"/>
       </geometry>
+      <material name="offwhite"/>
     </visual>
     <collision>
       <origin rpy="0 0 0" xyz="0 0 ${-table_inertia_z/2}"/>
       <geometry>
-        <xacro:if value="${collision_geometry == 'box'}">
-          <box size="1.5 2.0 0.05"/>
-        </xacro:if>
-        <xacro:if value="${collision_geometry == 'cylinder'}">
-          <cylinder radius="0.3" length="0.03" />
-        </xacro:if>
+        <box size="${wall_inertia_x} ${wall_inertia_y} ${wall_inertia_z}"/>
       </geometry>
     </collision>
-    <xacro:box_inertial x="${table_inertia_x}" y="${table_inertia_y}" z="${table_inertia_z}"  m="${table_mass}">
+    <xacro:box_inertial x="${wall_inertia_x}" y="${wall_inertia_y}" z="${wall_inertia_z}"  m="${wall_mass}">
       <origin rpy="0 0 0" xyz="0 0 ${-table_inertia_z/2}"/>
     </xacro:box_inertial>
