Commit message: updated urdfs for sand-gym UR%e

File: urdf/sand_gym_wooden_box_macro.urdf.xacro (robot description, xacro)
@@ -4,5 +4,5 @@
         <link name="${tf_prefix}wooden_box_base_link">
             <visual>
-                <origin xyz="0 0 0" rpy="0 0 0" />
+                <origin xyz="0 0 0" rpy="0 0 -1.57" />
                 <geometry>
                     <!-- Using STL for visual instead of DAE (Looks better :) ) -->
@@ -14,5 +14,5 @@
             </visual>
             <collision>
-                <origin xyz="0 0 0" rpy="0 0 0" />
+                <origin xyz="0 0 0" rpy="0 0 -1.57" />
                 <geometry>
                     <mesh filename="package://ur_description/meshes/collision/wooden_box.stl" scale="0.01 0.01 0.01"/>
@@ -21,5 +21,5 @@
             <inertial>
                 <mass value="0.2"/>
-                <origin xyz="0 0 0" rpy="0 0 0"/>
+                <origin xyz="0 0 0" rpy="0 0 -1.57"/>
                 <inertia ixx="0.001" ixy="0" ixz="0" iyy="0.001" iyz="0" izz="0.001"/>
             </inertial>

File: urdf/ur.urdf.xacro (robot description, xacro)
@@ -157,5 +157,5 @@
         parent="world"
       >
-        <origin xyz="0.0 0.9 0.0475" rpy="0 0 0"/>
+        <origin xyz="0.0 0.55 0.0475" rpy="0 0 1.57"/>
     </xacro:wooden_box>
 </xacro:if>
