Commit message: Added virtual gripper grasp point and ur5 calibration of real robot

File: urdf/ur_macro.xacro (robot description, xacro)
@@ -363,4 +363,19 @@
       <child link="${prefix}tool0"/>
     </joint>
+    <!-- Virtual Grasp Point Link -->
+    <link name="${prefix}gripper_grasp_point">
+    </link>
+    <!-- Virtual Grasp Point Fixed Joint -->
+    <joint name="${prefix}gripper_grasp_point_joint" type="fixed">
+      <parent link="tool0"/>
+      <child link="${prefix}gripper_grasp_point"/>
+      <!-- Center between finger tips -->
+      <!-- Matching the table origin -->
+      <!--<origin rpy="1.570796325 0 -1.570796325" xyz="${0.213-0.024/2} 0 0"/>-->
+      <!-- Matching the convention -->
+      <!--z offset closed gripper from base to fingertip 162.8mm (for rg2_ft its 220 + 25 for the quick changer) + force torque sensor 35mm-->
+      <origin rpy="0 0 0" xyz="0 0 0.279"/>
+      <!--<limit effort="0" lower="0" upper="0" velocity="0"/>-->
+    </joint>
   </xacro:macro>
 </robot>

Commit message: Changed virtual grasp point to Robotiq 2f-85 gripper

File: urdf/ur_macro.xacro (robot description, xacro)
@@ -374,6 +374,7 @@
       <!--<origin rpy="1.570796325 0 -1.570796325" xyz="${0.213-0.024/2} 0 0"/>-->
       <!-- Matching the convention -->
-      <!--z offset closed gripper from base to fingertip 162.8mm (for rg2_ft its 220 + 25 for the quick changer) + force torque sensor 35mm-->
-      <origin rpy="0 0 0" xyz="0 0 0.279"/>
+      <!--z offset closed OnRobot RG2-FT gripper from base to fingertip 220 + quick changer 25 + force torque sensor 35mm = 280 mm-->
+      <!--z offset closed Robotiq gripper from base to fingertip 162.8mm + force torque sensor 35mm-->
+      <origin rpy="0 0 0" xyz="0 0 0.1978"/>
       <!--<limit effort="0" lower="0" upper="0" velocity="0"/>-->
     </joint>

Commit message: Shortened virtual grasp point, because ft-sensor was removed

File: urdf/ur_macro.xacro (robot description, xacro)
@@ -376,5 +376,5 @@
       <!--z offset closed OnRobot RG2-FT gripper from base to fingertip 220 + quick changer 25 + force torque sensor 35mm = 280 mm-->
       <!--z offset closed Robotiq gripper from base to fingertip 162.8mm + force torque sensor 35mm-->
-      <origin rpy="0 0 0" xyz="0 0 0.1978"/>
+      <origin rpy="0 0 0" xyz="0 0 0.1628"/>
       <!--<limit effort="0" lower="0" upper="0" velocity="0"/>-->
     </joint>

Commit message: Joint Trajectory Controller Config Change

File: urdf/ur_macro.xacro (robot description, xacro)
@@ -400,5 +400,5 @@
       <parent link="tool0"/>
       <child link="${tf_prefix}custom_gripper_grasp_point"/>
-      <origin rpy="0 0 0" xyz="0 0 0.150"/>
+      <origin rpy="0 0 -0.785413110" xyz="0 0 0.150"/>
     </joint>
   </xacro:macro>
