Commit message: Calibrating UR3e Camera Mount

File: urdf/suction_gripper_macro.urdf.xacro (robot description, xacro)
@@ -32,6 +32,5 @@
         </joint>
         <!-- Mount reference frame positioned -31.5mm in x relative to parent -->
-        <link name="${tf_prefix}mount_reference">
-            <!-- Empty link for reference frame only -->
+        <!-- <link name="${tf_prefix}mount_reference">
         </link>
         <joint name="${tf_prefix}mount_reference_joint" type="fixed">
@@ -39,5 +38,5 @@
             <child link="${tf_prefix}mount_reference"/>
             <origin xyz="-0.0315 0 0.007" rpy="0 0 0"/>
-        </joint>
+        </joint> -->
         <!-- Gripper tip link at the center bottom of the gripper -->
         <link name="${tf_prefix}ecpmi_gripper_tip">

File: urdf/ur.urdf.xacro (robot description, xacro)
@@ -200,4 +200,5 @@
   </xacro:if>
   <!-- UR3e in-hand camera mount -->
+   <!-- <origin xyz="0.0 0.0 -0.013" rpy="0 0 0"/> -->
   <xacro:if value="$(arg use_ur3e_camera_mount)">
     <xacro:ur3e_inhand_camera_mount

File: urdf/ur3e_inhand_camera_mount_macro.urdf.xacro (robot description, xacro)
@@ -27,4 +27,15 @@
             </inertial>
         </link>
+        <!-- Mount reference frame positioned -31.5mm in x relative to parent -->
+        <link name="${tf_prefix}mount_reference">
+        </link>
+        <!-- Original -->
+        <!-- <origin xyz="-0.0315 0 0.007" rpy="0 0 0"/> -->
+        <!-- <origin xyz="-0.03305 0 0.007 " rpy="0 0 0"/> -->
+        <joint name="${tf_prefix}mount_reference_joint" type="fixed">
+            <parent link="${parent}"/>
+            <child link="${tf_prefix}mount_reference"/>
+             <origin xyz="-0.03305 0 0.007 " rpy="0 0 0"/>
+        </joint>
         <!-- Join the camera mount to the parent link (tool0) -->
         <joint name="${tf_prefix}ur3e_inhand_camera_mount_joint" type="fixed">
@@ -36,5 +47,4 @@
         <link name="${tf_prefix}camera_mount_reference">
         </link>
-       <!-- <origin xyz="0.128610 -0.000620291 0.025456" rpy="0.261826 0.000000 -1.570917"/> -->
         <joint name="${tf_prefix}camera_mount_reference_joint" type="fixed">
             <parent link="${tf_prefix}mount_reference"/>
