Commit message: Added collision objects table, top, wall with table_macro

File: urdf/ur.urdf.xacro (robot description, xacro)
@@ -5,4 +5,5 @@
    <!-- import main macro -->
    <xacro:include filename="$(find ur_description)/urdf/ur_macro.xacro"/>
+   <xacro:include filename="$(find ur_description)/urdf/table_macro.xacro"/>
    <!-- possible 'ur_type' values: ur3, ur3e, ur5, ur5e, ur10, ur10e, ur16e -->
    <!-- the default value should raise an error in case this was called without defining the type -->
@@ -34,4 +35,6 @@
    <xacro:arg name="tool_device_name" default="/tmp/ttyUR" />
    <xacro:arg name="tool_tcp_port" default="54321" />
+   <!-- Table parameters -->
+   <xacro:arg name="physical_params_table" default="$(find ur_description)/config/table/physical_parameters_table.yaml"/>
      <!-- Simulation parameters -->
    <xacro:arg name="use_fake_hardware" default="false" />
@@ -40,4 +43,6 @@
    <xacro:arg name="sim_ignition" default="false" />
    <xacro:arg name="simulation_controllers" default="" />
+   <!-- Flag to preserve fixed joints and prevent lumping when generating SDF for Gazebo -->
+   <xacro:arg name="gazebo_preserve_fixed_joint_arg" default="false"/>
    <!-- initial position for simulations (Fake Hardware, Gazebo, Ignition) -->
    <xacro:arg name="initial_positions_file" default="$(find ur_description)/config/initial_positions.yaml"/>
@@ -46,4 +51,44 @@
    <!-- create link fixed to the "world" -->
    <link name="world" />
+   <!-- Load configuration data from the provided .yaml files -->
+    <xacro:read_table_data
+      physical_parameters_table_file="$(arg physical_params_table)"
+    />
+   <!-- table -->
+   <xacro:table_attach
+     prefix="$(arg prefix)"
+     name="table"
+     parent="world"
+     sim_gazebo="$(arg sim_gazebo)"
+     sim_ignition="$(arg sim_ignition)"
+     gazebo_preserve_fixed_joint="$(arg gazebo_preserve_fixed_joint_arg)"
+     physical_parameters_table_file="$(arg physical_params_table)"
+     >
+     <origin xyz="-0.232 0.415 0" rpy="0 0 0"/>
+   </xacro:table_attach>
+   <!-- top -->
+   <xacro:table_attach
+     prefix="$(arg prefix)"
+     name="top"
+     parent="world"
+     sim_gazebo="$(arg sim_gazebo)"
+     sim_ignition="$(arg sim_ignition)"
+     gazebo_preserve_fixed_joint="$(arg gazebo_preserve_fixed_joint_arg)"
+     physical_parameters_table_file="$(arg physical_params_table)"
+     >
+     <origin xyz="-0.232 0.415 0.7" rpy="0 0 0"/>
+   </xacro:table_attach>
+    <!-- wall -->
+   <xacro:table_attach
+     prefix="$(arg prefix)"
+     name="wall"
+     parent="world"
+     sim_gazebo="$(arg sim_gazebo)"
+     sim_ignition="$(arg sim_ignition)"
+     gazebo_preserve_fixed_joint="$(arg gazebo_preserve_fixed_joint_arg)"
+     physical_parameters_table_file="$(arg physical_params_table)"
+     >
+     <origin xyz="-0.618 0.0 0.35" rpy="0 1.57 0"/>
+   </xacro:table_attach>
    <!-- arm -->
    <xacro:ur_robot

Commit message: added gripper urdf to the existing arm urdf

File: urdf/ur.urdf.xacro (robot description, xacro)
@@ -6,4 +6,5 @@
    <xacro:include filename="$(find ur_description)/urdf/ur_macro.xacro"/>
    <xacro:include filename="$(find ur_description)/urdf/table_macro.xacro"/>
+   <xacro:include filename="$(find ur_description)/urdf/robotiq_85_gripper_macro.urdf.xacro"/>
    <!-- possible 'ur_type' values: ur3, ur3e, ur5, ur5e, ur10, ur10e, ur16e -->
    <!-- the default value should raise an error in case this was called without defining the type -->
@@ -91,4 +92,11 @@
      <origin xyz="-0.618 0.0 0.35" rpy="0 1.57 0"/>
    </xacro:table_attach>
+   <!-- gripper -->
+   <xacro:robotiq_85_gripper
+     prefix="$(arg prefix)"
+     parent="tool0"
+     >
+     <origin xyz="0.0 0.0 0.0" rpy="-1.57 -1.57 0"/>
+   </xacro:robotiq_85_gripper>
    <!-- arm -->
    <xacro:ur_robot

Commit message: Repair Demo

File: urdf/ur.urdf.xacro (robot description, xacro)
@@ -66,4 +66,9 @@
    <!-- create link fixed to the "world" -->
    <link name="world" />
+   <!-- create link fixed to the "world" -->
+   <!--<link name="world">
+    <origin xyz="0 0 0" rpy="0 0 1.57"/>
+   </link>
+  -->
    <!-- Load configuration data from the provided .yaml files -->
     <xacro:read_table_data
@@ -166,5 +171,5 @@
      script_sender_port="$(arg script_sender_port)"
      trajectory_port="$(arg trajectory_port)" -->
-     <origin xyz="0 0 0" rpy="0 0 0" />          <!-- position robot in the world -->
+     <origin xyz="0 0 0" rpy="0 0 1.57" />          <!-- position robot in the world -->
    </xacro:ur_robot>
    <xacro:if value="$(arg sim_gazebo)">

Commit message: Making changes for the UR5e Setup

File: urdf/ur.urdf.xacro (robot description, xacro)
@@ -11,7 +11,15 @@
    <xacro:include filename="$(find ur_description)/urdf/table_collision_macro.xacro"/>
    <xacro:include filename="$(find ur_description)/urdf/robotiq_gripper_macro.urdf.xacro"/>
+   <xacro:include filename="$(find ur_description)/urdf/custom_gripper_macro.urdf.xacro"/>
+    <xacro:include filename="$(find ur_description)/urdf/sand_gym_wooden_box_macro.urdf.xacro"/>
    <!-- possible 'ur_type' values: ur3, ur3e, ur5, ur5e, ur10, ur10e, ur16e, ur20, ur30 -->
    <!-- the default value should raise an error in case this was called without defining the type -->
    <xacro:arg name="ur_type" default="ur5x"/>
+   <xacro:arg name="is_ur3_setup" default="false"/>
+   <xacro:arg name="is_ur5_setup" default="false"/>
+   <xacro:arg name="is_ur5e_setup" default="false"/>
+   <xacro:property name="is_ur3_setup" value="$(arg is_ur3_setup)" />
+   <xacro:property name="is_ur5_setup" value="$(arg is_ur5_setup)" />
+   <xacro:property name="is_ur5e_setup" value="$(arg is_ur5e_setup)" />
    <!-- parameters -->
    <xacro:arg name="tf_prefix" default="" />
@@ -46,7 +54,10 @@
    <xacro:arg name="tool_tcp_port" default="54321" />
    <!-- Flag to use the Gripper or just the UR5  -->
-   <xacro:arg name="use_gripper" default="true" />
+   <xacro:arg name="use_gripper" default="false" />
+   <!-- Flag to choose between custom gripper and robotiq gripper -->
+   <xacro:arg name="use_custom_gripper" default="false" />
    <!-- Table parameters -->
-   <xacro:arg name="physical_params_table" default="$(find ur_description)/config/table/physical_parameters_table.yaml"/>
+   <xacro:arg name="physical_params_ur5_table" default="$(find ur_description)/config/table/physical_parameters_ur5_table.yaml"/>
+   <xacro:arg name="physical_params_ur5e_table" default="$(find ur_description)/config/table/physical_parameters_ur5e_table.yaml"/>
    <xacro:arg name="ring_beam_height" default="1.0"/>
      <!-- Simulation parameters -->
@@ -59,5 +70,5 @@
    <xacro:arg name="gazebo_preserve_fixed_joint_arg" default="false"/>
    <!-- Flag to use the Gripper or just the UR5  -->
-   <xacro:arg name="use_gripper" default="true" />
+   <xacro:arg name="use_gripper" default="false" />
    <!-- initial position for simulations (Fake Hardware, Gazebo, Ignition) -->
    <xacro:arg name="initial_positions_file" default="$(find ur_description)/config/initial_positions.yaml"/>
@@ -71,8 +82,9 @@
    </link>
   -->
-   <!-- Load configuration data from the provided .yaml files -->
-    <xacro:read_table_data
-      physical_parameters_table_file="$(arg physical_params_table)"
-    />
+<xacro:if value="${is_ur5_setup}">
+    <!-- Load configuration data from the provided .yaml files -->
+  <xacro:read_table_data
+    physical_parameters_table_file="$(arg physical_params_ur5_table)"
+  />
    <!-- table -->
    <xacro:table_attach
@@ -83,53 +95,91 @@
      sim_ignition="$(arg sim_ignition)"
      gazebo_preserve_fixed_joint="$(arg gazebo_preserve_fixed_joint_arg)"
-     physical_parameters_table_file="$(arg physical_params_table)"
+     physical_parameters_table_file="$(arg physical_params_ur5_table)"
      >
      <origin xyz="-0.232 0.415 0" rpy="0 0 0"/>
    </xacro:table_attach>
-   <!-- ringlight -->
-   <xacro:ringlight_attach
+    <!-- ringlight -->
+    <xacro:ringlight_attach
+      tf_prefix="$(arg tf_prefix)"
+      name="ringlight"
+      parent="world"
+      sim_gazebo="$(arg sim_gazebo)"
+      sim_ignition="$(arg sim_ignition)"
+      gazebo_preserve_fixed_joint="$(arg gazebo_preserve_fixed_joint_arg)"
+      physical_parameters_table_file="$(arg physical_params_ur5_table)"
+      >
+      <origin xyz="-0.232 0.415 $(arg ring_beam_height)" rpy="0 0 0"/>
+    </xacro:ringlight_attach>
+    <!-- beam -->
+    <xacro:beam_attach
+      tf_prefix="$(arg tf_prefix)"
+      name="beam"
+      parent="world"
+      sim_gazebo="$(arg sim_gazebo)"
+      sim_ignition="$(arg sim_ignition)"
+      gazebo_preserve_fixed_joint="$(arg gazebo_preserve_fixed_joint_arg)"
+      physical_parameters_table_file="$(arg physical_params_ur5_table)"
+      >
+      <origin xyz="-0.518 0.415 $(arg ring_beam_height)" rpy="0 0 0"/>
+    </xacro:beam_attach>
+      <!-- wall -->
+    <xacro:wall_attach
+      tf_prefix="$(arg tf_prefix)"
+      name="wall"
+      parent="world"
+      sim_gazebo="$(arg sim_gazebo)"
+      sim_ignition="$(arg sim_ignition)"
+      gazebo_preserve_fixed_joint="$(arg gazebo_preserve_fixed_joint_arg)"
+      physical_parameters_table_file="$(arg physical_params_ur5_table)"
+      >
+      <origin xyz="-0.618 0.0 0.35" rpy="0 1.57 0"/>
+    </xacro:wall_attach>
+  </xacro:if>
+<xacro:if value="${is_ur5e_setup}">
+    <!-- Load configuration data from the provided .yaml files -->
+  <xacro:read_table_data
+    physical_parameters_table_file="$(arg physical_params_ur5e_table)"
+  />
+   <!-- table -->
+   <xacro:table_attach
      tf_prefix="$(arg tf_prefix)"
-     name="ringlight"
+     name="table"
      parent="world"
      sim_gazebo="$(arg sim_gazebo)"
      sim_ignition="$(arg sim_ignition)"
      gazebo_preserve_fixed_joint="$(arg gazebo_preserve_fixed_joint_arg)"
-     physical_parameters_table_file="$(arg physical_params_table)"
+     physical_parameters_table_file="$(arg physical_params_ur5e_table)"
      >
-     <origin xyz="-0.232 0.415 $(arg ring_beam_height)" rpy="0 0 0"/>
-   </xacro:ringlight_attach>
-   <!-- beam -->
-   <xacro:beam_attach
-     tf_prefix="$(arg tf_prefix)"
-     name="beam"
-     parent="world"
-     sim_gazebo="$(arg sim_gazebo)"
-     sim_ignition="$(arg sim_ignition)"
-     gazebo_preserve_fixed_joint="$(arg gazebo_preserve_fixed_joint_arg)"
-     physical_parameters_table_file="$(arg physical_params_table)"
-     >
-     <origin xyz="-0.518 0.415 $(arg ring_beam_height)" rpy="0 0 0"/>
-   </xacro:beam_attach>
-    <!-- wall -->
-   <xacro:wall_attach
-     tf_prefix="$(arg tf_prefix)"
-     name="wall"
-     parent="world"
-     sim_gazebo="$(arg sim_gazebo)"
-     sim_ignition="$(arg sim_ignition)"
-     gazebo_preserve_fixed_joint="$(arg gazebo_preserve_fixed_joint_arg)"
-     physical_parameters_table_file="$(arg physical_params_table)"
-     >
-     <origin xyz="-0.618 0.0 0.35" rpy="0 1.57 0"/>
-   </xacro:wall_attach>
-   <!-- gripper -->
-   <xacro:if value="$(arg use_gripper)">
-   <xacro:robotiq_gripper
-     tf_prefix="$(arg tf_prefix)"
-     parent="tool0"
-     >
-     <origin xyz="0.0 0.0 0.0" rpy="0 0 0"/>
-   </xacro:robotiq_gripper>
-   </xacro:if>
+     <origin xyz="0 0.2 0" rpy="0 0 0"/>
+   </xacro:table_attach>
+   <xacro:wooden_box
+        tf_prefix="$(arg tf_prefix)"
+        parent="world"
+      >
+        <origin xyz="0.0 0.9 0.0475" rpy="0 0 0"/>
+    </xacro:wooden_box>
+</xacro:if>
+  <!-- robotiq gripper -->
+  <xacro:if value="$(arg use_gripper)">
+    <xacro:unless value="$(arg use_custom_gripper)">
+      <xacro:robotiq_gripper
+        tf_prefix="$(arg tf_prefix)"
+        parent="tool0"
+      >
+        <origin xyz="0.0 0.0 0.0" rpy="0 0 0"/>
+      </xacro:robotiq_gripper>
+    </xacro:unless>
+  </xacro:if>
+  <!-- custom gripper (sand_gym) -->
+  <xacro:if value="$(arg use_custom_gripper)">
+    <xacro:unless value="$(arg use_gripper)">
+      <xacro:custom_gripper
+        tf_prefix="$(arg tf_prefix)"
+        parent="tool0"
+      >
+        <origin xyz="0.0 0.0 0.0" rpy="0 0 0"/>
+      </xacro:custom_gripper>
+    </xacro:unless>
+  </xacro:if>
    <!-- arm -->
    <xacro:ur_robot
@@ -171,5 +221,5 @@
      script_sender_port="$(arg script_sender_port)"
      trajectory_port="$(arg trajectory_port)" -->
-     <origin xyz="0 0 0" rpy="0 0 1.57" />          <!-- position robot in the world -->
+     <origin xyz="0 0 0" rpy="0 0 0" />          <!-- position robot in the world -->
    </xacro:ur_robot>
    <xacro:if value="$(arg sim_gazebo)">

File: urdf/ur_macro.xacro (robot description, xacro)
@@ -381,4 +381,7 @@
     <link name="${tf_prefix}gripper_grasp_point">
     </link>
+    <!-- Virtual Custom Gripper Grasp Point Link -->
+    <link name="${tf_prefix}custom_gripper_grasp_point">
+    </link>
     <!-- Virtual Grasp Point Fixed Joint -->
     <joint name="${tf_prefix}gripper_grasp_point_joint" type="fixed">
@@ -394,4 +397,9 @@
       <!--<limit effort="0" lower="0" upper="0" velocity="0"/>-->
     </joint>
+    <joint name="${tf_prefix}custom_gripper_grasp_point_joint" type="fixed">
+      <parent link="tool0"/>
+      <child link="${tf_prefix}custom_gripper_grasp_point"/>
+      <origin rpy="0 0 0" xyz="0 0 0.150"/>
+    </joint>
   </xacro:macro>
 </robot>

Commit message: UR3e changes along with Suction Gripper

File: urdf/ur.urdf.xacro (robot description, xacro)
@@ -12,12 +12,14 @@
    <xacro:include filename="$(find ur_description)/urdf/robotiq_gripper_macro.urdf.xacro"/>
    <xacro:include filename="$(find ur_description)/urdf/custom_gripper_macro.urdf.xacro"/>
+   <xacro:include filename="$(find ur_description)/urdf/suction_gripper_macro.urdf.xacro"/>
+   <xacro:include filename="$(find ur_description)/urdf/ur3e_inhand_camera_mount_macro.urdf.xacro"/>
     <xacro:include filename="$(find ur_description)/urdf/sand_gym_wooden_box_macro.urdf.xacro"/>
    <!-- possible 'ur_type' values: ur3, ur3e, ur5, ur5e, ur10, ur10e, ur16e, ur20, ur30 -->
    <!-- the default value should raise an error in case this was called without defining the type -->
    <xacro:arg name="ur_type" default="ur5x"/>
-   <xacro:arg name="is_ur3_setup" default="false"/>
+   <xacro:arg name="is_ur3e_setup" default="false"/>
    <xacro:arg name="is_ur5_setup" default="false"/>
    <xacro:arg name="is_ur5e_setup" default="false"/>
-   <xacro:property name="is_ur3_setup" value="$(arg is_ur3_setup)" />
+   <xacro:property name="is_ur3e_setup" value="$(arg is_ur3e_setup)" />
    <xacro:property name="is_ur5_setup" value="$(arg is_ur5_setup)" />
    <xacro:property name="is_ur5e_setup" value="$(arg is_ur5e_setup)" />
@@ -57,4 +59,8 @@
    <!-- Flag to choose between custom gripper and robotiq gripper -->
    <xacro:arg name="use_custom_gripper" default="false" />
+   <!-- Flag to choose suction gripper -->
+   <xacro:arg name="use_suction_gripper" default="false" />
+   <!-- Flag to use UR3e in-hand camera mount -->
+   <xacro:arg name="use_ur3e_camera_mount" default="true" />
    <!-- Table parameters -->
    <xacro:arg name="physical_params_ur5_table" default="$(find ur_description)/config/table/physical_parameters_ur5_table.yaml"/>
@@ -182,4 +188,24 @@
     </xacro:unless>
   </xacro:if>
+  <!-- suction gripper -->
+  <xacro:if value="$(arg use_suction_gripper)">
+    <xacro:unless value="$(arg use_gripper)">
+      <xacro:ecpmi_gripper
+        tf_prefix="$(arg tf_prefix)"
+        parent="tool0"
+      >
+        <origin xyz="0.0 0.0 0.0" rpy="0 0 2.36"/>
+      </xacro:ecpmi_gripper>
+    </xacro:unless>
+  </xacro:if>
+  <!-- UR3e in-hand camera mount -->
+  <xacro:if value="$(arg use_ur3e_camera_mount)">
+    <xacro:ur3e_inhand_camera_mount
+      tf_prefix="$(arg tf_prefix)"
+      parent="tool0"
+    >
+      <origin xyz="0.0 0.0 -0.013" rpy="0 0 0"/>
+    </xacro:ur3e_inhand_camera_mount>
+  </xacro:if>
    <!-- arm -->
    <xacro:ur_robot

File: urdf/ur_macro.xacro (robot description, xacro)
@@ -384,4 +384,7 @@
     <link name="${tf_prefix}custom_gripper_grasp_point">
     </link>
+    <!-- Virtual ECPMI Gripper Grasp Point Link -->
+    <link name="${tf_prefix}ecpmi_gripper_grasp_point">
+    </link>
     <!-- Virtual Grasp Point Fixed Joint -->
     <joint name="${tf_prefix}gripper_grasp_point_joint" type="fixed">
@@ -402,4 +405,16 @@
       <origin rpy="0 0 -0.785413110" xyz="0 0 0.150"/>
     </joint>
+    <joint name="${tf_prefix}ecpmi_gripper_grasp_point_joint" type="fixed">
+      <parent link="tool0"/>
+      <child link="${tf_prefix}ecpmi_gripper_grasp_point"/>
+      <!-- ECPMI suction gripper grasp point at tip -->
+      <origin rpy="0 0 0" xyz="0 0 0.107"/>
+    </joint>
+    <!-- Joint connecting wrist_3_link to camera mount -->
+    <!-- <joint name="${tf_prefix}ur3e_inhand_camera_mount_joint" type="fixed">
+      <parent link="${tf_prefix}wrist_3_link"/>
+      <child link="${tf_prefix}ur3e_inhand_camera_mount"/>
+      <origin xyz="0 0 0" rpy="0 0 0"/>
+    </joint> -->
   </xacro:macro>
 </robot>

Commit message: updating changes for RIGs Demo

File: urdf/ur.urdf.xacro (robot description, xacro)
@@ -15,8 +15,9 @@
    <xacro:include filename="$(find ur_description)/urdf/ur3e_inhand_camera_mount_macro.urdf.xacro"/>
     <xacro:include filename="$(find ur_description)/urdf/sand_gym_wooden_box_macro.urdf.xacro"/>
+    <xacro:include filename="$(find ur_description)/urdf/ur_llm_wooden_box_macro.urdf.xacro"/>
    <!-- possible 'ur_type' values: ur3, ur3e, ur5, ur5e, ur10, ur10e, ur16e, ur20, ur30 -->
    <!-- the default value should raise an error in case this was called without defining the type -->
    <xacro:arg name="ur_type" default="ur5x"/>
-   <xacro:arg name="is_ur3e_setup" default="false"/>
+   <xacro:arg name="is_ur3e_setup" default="true"/>
    <xacro:arg name="is_ur5_setup" default="false"/>
    <xacro:arg name="is_ur5e_setup" default="false"/>
@@ -66,4 +67,5 @@
    <xacro:arg name="physical_params_ur5_table" default="$(find ur_description)/config/table/physical_parameters_ur5_table.yaml"/>
    <xacro:arg name="physical_params_ur5e_table" default="$(find ur_description)/config/table/physical_parameters_ur5e_table.yaml"/>
+   <xacro:arg name="physical_params_ur3e_table" default="$(find ur_description)/config/table/physical_parameters_ur3e_table.yaml"/>
    <xacro:arg name="ring_beam_height" default="1.0"/>
      <!-- Simulation parameters -->
@@ -166,4 +168,40 @@
     </xacro:wooden_box>
 </xacro:if>
+<xacro:if value="${is_ur3e_setup}">
+      <!-- Load configuration data from the provided .yaml files -->
+    <xacro:read_table_data
+      physical_parameters_table_file="$(arg physical_params_ur3e_table)"
+    />
+    <!-- table -->
+    <xacro:table_attach
+      tf_prefix="$(arg tf_prefix)"
+      name="table"
+      parent="world"
+      sim_gazebo="$(arg sim_gazebo)"
+      sim_ignition="$(arg sim_ignition)"
+      gazebo_preserve_fixed_joint="$(arg gazebo_preserve_fixed_joint_arg)"
+      physical_parameters_table_file="$(arg physical_params_ur5e_table)"
+      >
+      <origin xyz="0 0 0" rpy="0 0 0"/>
+    </xacro:table_attach>
+    <!-- wall -->
+    <xacro:wall_attach
+      tf_prefix="$(arg tf_prefix)"
+      name="wall"
+      parent="world"
+      sim_gazebo="$(arg sim_gazebo)"
+      sim_ignition="$(arg sim_ignition)"
+      gazebo_preserve_fixed_joint="$(arg gazebo_preserve_fixed_joint_arg)"
+      physical_parameters_table_file="$(arg physical_params_ur3e_table)"
+      >
+      <origin xyz="0.4 0.0 0.35" rpy="0 1.57 0"/>
+    </xacro:wall_attach>
+    <xacro:ur_llm_wooden_box
+        tf_prefix="$(arg tf_prefix)"
+        parent="world"
+      >
+        <origin xyz="-0.28 0.21 0.08" rpy="0 0 0"/>
+    </xacro:ur_llm_wooden_box>
+  </xacro:if>
   <!-- robotiq gripper -->
   <xacro:if value="$(arg use_gripper)">
