Commit message: geo sem running on UR5e properly

File: urdf/robotiq_gripper_macro.urdf.xacro (robot description, xacro)
@@ -7,5 +7,5 @@
         <xacro:robotiq_gripper_ros2_control
           name="robotiq_gripper_control"
-          com_port="/dev/ttyUSB0"/>
+          com_port="/tmp/ttyUR"/>
         <link name="${tf_prefix}robotiq_85_base_link">
             <visual>

File: urdf/ur.urdf.xacro (robot description, xacro)
@@ -161,5 +161,5 @@
      script_sender_port="$(arg script_sender_port)"
      trajectory_port="$(arg trajectory_port)" -->
-     <origin xyz="0 0 0.72" rpy="0 0 1.570796327" />          <!-- position robot in the world -->
+     <origin xyz="0 0 0" rpy="0 0 0" />          <!-- world coincides with the robot base -->
    </xacro:ur_robot>
    <xacro:if value="$(arg sim_gazebo)">
