Commit message: xacro.load_yaml update

File: urdf/inc/table_common.xacro (robot description, xacro)
@@ -3,5 +3,5 @@
   <xacro:macro name="read_table_data" params="physical_parameters_table_file">
     <!-- Read .yaml files from disk, load content into properties -->
-    <xacro:property name="config_physical_parameters_table" value="${load_yaml(physical_parameters_table_file)}"/>
+    <xacro:property name="config_physical_parameters_table" value="${xacro.load_yaml(physical_parameters_table_file)}"/>
     <!-- Extract subsections from yaml dictionaries -->
     <xacro:property name="sec_inertia_parameters" value="${config_physical_parameters_table['inertia_parameters']}" />
